Commit message: Numerous fixes

File: urdf/two_link.urdf (robot description, URDF)
Before this commit: robot reacher, 5 links, 4 joints
Joints:
- joint joint0: limit lower=-3.00000 upper=3.00000 effort=20.0 velocity=5.0 -> effort=20.0 velocity=5.0; type revolute -> continuous

Commit message: Changes to the pybullet environment

File: urdf/two_link.urdf (robot description, URDF)
Before this commit: robot reacher, 5 links, 4 joints
Joints:
- joint joint0: limit effort=20.0 velocity=5.0 -> effort=20.0 velocity=15.0
- joint joint1: limit lower=-3.00000 upper=3.00000 effort=20.0 velocity=5.0 -> lower=-3.00000 upper=3.00000 effort=20.0 velocity=15.0

Commit message: Reacher environment pybullet

File: urdf/two_link.urdf (robot description, URDF)
Before this commit: robot reacher, 5 links, 4 joints
Joints:
- joint joint0: limit effort=20.0 velocity=15.0 -> effort=20.0 velocity=5.0
- joint joint1: limit lower=-3.00000 upper=3.00000 effort=20.0 velocity=15.0 -> lower=-3.00000 upper=3.00000 effort=20.0 velocity=5.0
