Commit message: Tested Gym wrapper with urdf file

File: urdf/seven_link.urdf (robot description, URDF)
Before this commit: robot reacher_seven_links, 15 links, 14 joints
Joints:
- joint joint_revolute_1: limit lower=-3.05 upper=3.05 effort=200 velocity=5.0 -> lower=-3.05 upper=3.05 effort=80 velocity=5.0
- joint joint_revolute_2: limit lower=-3.05 upper=3.05 effort=1 velocity=5.0 -> lower=-3.05 upper=3.05 effort=80 velocity=5.0
- joint joint_revolute_3: limit lower=-3.05 upper=3.05 effort=1 velocity=5.0 -> lower=-3.05 upper=3.05 effort=80 velocity=5.0
- joint joint_revolute_4: limit lower=-3.05 upper=3.05 effort=1 velocity=5.0 -> lower=-3.05 upper=3.05 effort=80 velocity=5.0
- joint joint_revolute_5: limit lower=-3.05 upper=3.05 effort=1 velocity=5.0 -> lower=-3.05 upper=3.05 effort=80 velocity=5.0
- joint joint_revolute_6: limit lower=-3.05 upper=3.05 effort=1 velocity=5.0 -> lower=-3.05 upper=3.05 effort=80 velocity=5.0

File: urdf/seven_link.urdf.xacro (robot description, xacro)
@@ -78,10 +78,10 @@
 	<xacro:link_group link_number="5"/>
 	<xacro:link_group link_number="6"/>
-	<xacro:joint_group angle="3.05" joint_number="0" force="200"/>
-	<xacro:joint_group angle="3.05" joint_number="1" force="1"/>
-	<xacro:joint_group angle="3.05" joint_number="2" force="1"/>
-	<xacro:joint_group angle="3.05" joint_number="3" force="1"/>
-	<xacro:joint_group angle="3.05" joint_number="4" force="1"/>
-	<xacro:joint_group angle="3.05" joint_number="5" force="1"/>
+	<xacro:joint_group angle="3.05" joint_number="0" force="80"/>
+	<xacro:joint_group angle="3.05" joint_number="1" force="80"/>
+	<xacro:joint_group angle="3.05" joint_number="2" force="80"/>
+	<xacro:joint_group angle="3.05" joint_number="3" force="80"/>
+	<xacro:joint_group angle="3.05" joint_number="4" force="80"/>
+	<xacro:joint_group angle="3.05" joint_number="5" force="80"/>
 	<link name="fingertip">
 		<inertial>
